File: TEEKeeper_Shield/TEEKeeper - Kicad Project/Digital_PCB.kicad_sch (KiCad schematic)
At the start: 7 parts

Commit message: Minor changes
Parts:
- R12, R9: value 10 -> 0
Other:
- note added: "R9, R12 are zero-value resistors. Add appropriate resistors if you experience noise issueson the SPI lines."
Changed lines of the file:
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@@
+		)
+	)
+	(text "R9, R12 are zero-value resistors. \nAdd appropriate resistors if you \nexperience noise issueson the SPI lines."
+		(exclude_from_sim no)
+		(at 209.55 122.174 0)
+		(effects
+			(font
+				(size 1.27 1.27)
+			)
+			(justify left)
 		)
 	)
@@
 			)
 		)
-		(property "Value" "10"
+		(property "Value" "0"
 			(at 191.77 91.4399 0)
 			(effects
@@
 			)
 		)
-		(property "Value" "10"
+		(property "Value" "0"
 			(at 156.21 91.4399 0)
 			(effects
