File: TEEKeeper_Shield/TEEKeeper - Kicad Project/System_Shiedl.kicad_sch (KiCad schematic)
At the start: 7 parts

Commit message: Resolved minor issues
Fixed broken / bad designed reference connections, fixed pcb courtyard and edges, general cleanup
Connections:
- net Digital_PCB/5V renamed 5V
- net 5V: no longer A1.5V4 (5V)
Changed lines of the file:
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@@
-	)
-	(junction
-		(at 191.77 147.32)
-		(diameter 0)
-		(color 0 0 0 0)
 	)
 	(junction
@@
 	)
 	(junction
-		(at 189.23 147.32)
-		(diameter 0)
-		(color 0 0 0 0)
-	)
-	(junction
 		(at 209.55 147.32)
 		(diameter 0)
@@
 	(wire
 		(pts
+			(xy 191.77 152.4) (xy 193.04 152.4)
+		)
+		(stroke
+			(width 0)
+			(type default)
+		)
+	)
+	(wire
+		(pts
 			(xy 71.12 66.04) (xy 100.33 66.04)
 		)
@@
 	(wire
 		(pts
-			(xy 236.22 156.21) (xy 189.23 156.21)
-		)
-		(stroke
-			(width 0)
-			(type default)
-		)
-	)
-	(wire
-		(pts
 			(xy 82.55 36.83) (xy 82.55 154.94)
 		)
@@
 	(wire
 		(pts
+			(xy 71.12 24.13) (xy 83.82 24.13)
+		)
+		(stroke
+			(width 0)
+			(type default)
+		)
+	)
+	(wire
+		(pts
 			(xy 137.16 162.56) (xy 129.54 162.56)
 		)
@@
 	(wire
 		(pts
+			(xy 189.23 156.21) (xy 190.5 156.21)
+		)
+		(stroke
+			(width 0)
+			(type default)
+		)
+	)
+	(wire
+		(pts
 			(xy 167.64 177.8) (xy 167.64 156.21)
 		)
@@
 	(wire
 		(pts
-			(xy 191.77 147.32) (xy 189.23 147.32)
-		)
-		(stroke
-			(width 0)
-			(type default)
-		)
-	)
-	(wire
-		(pts
 			(xy 80.01 39.37) (xy 80.01 157.48)
 		)
@@
 	(wire
 		(pts
-			(xy 236.22 24.13) (xy 236.22 156.21)
-		)
-		(stroke
-			(width 0)
-			(type default)
-		)
-	)
-	(wire
-		(pts
 			(xy 204.47 147.32) (xy 207.01 147.32)
 		)
@@
 	(wire
 		(pts
-			(xy 194.31 147.32) (xy 191.77 147.32)
-		)
-		(stroke
-			(width 0)
-			(type default)
-		)
-	)
-	(wire
-		(pts
 			(xy 207.01 153.67) (xy 207.01 147.32)
 		)
@@
 	(wire
 		(pts
+			(xy 191.77 147.32) (xy 191.77 152.4)
+		)
+		(stroke
+			(width 0)
+			(type default)
+		)
+	)
+	(wire
+		(pts
 			(xy 86.36 170.18) (xy 81.28 170.18)
 		)
@@
 		(pts
 			(xy 156.21 167.64) (xy 156.21 162.56)
-		)
-		(stroke
-			(width 0)
-			(type default)
-		)
-	)
-	(wire
-		(pts
-			(xy 71.12 24.13) (xy 236.22 24.13)
 		)
 		(stroke
@@
 			)
 		)
+	)
+	(global_label "5V"
+		(shape input)
+		(at 193.04 152.4 0)
+		(fields_autoplaced yes)
+		(effects
+			(font
+				(size 1.27 1.27)
+			)
+			(justify left)
+		)
+		(property "Intersheetrefs" "${INTERSHEET_REFS}"
+			(at 198.3233 152.4 0)
+			(effects
+				(font
+					(size 1.27 1.27)
+				)
+				(justify left)
+				(hide yes)
+			)
+		)
+	)
+	(global_label "5V"
+		(shape input)
+		(at 83.82 24.13 0)
+		(fields_autoplaced yes)
+		(effects
+			(font
+				(size 1.27 1.27)
+			)
+			(justify left)
+		)
+		(property "Intersheetrefs" "${INTERSHEET_REFS}"
+			(at 89.1033 24.13 0)
+			(effects
+				(font
+					(size 1.27 1.27)
+				)
+				(justify left)
+				(hide yes)
+			)
+		)
+	)
+	(global_label "5V"
+		(shape input)
+		(at 190.5 156.21 0)
+		(fields_autoplaced yes)
+		(effects
+			(font
+				(size 1.27 1.27)
+			)
+			(justify left)
+		)
+		(property "Intersheetrefs" "${INTERSHEET_REFS}"
+			(at 195.7833 156.21 0)
+			(effects
+				(font
+					(size 1.27 1.27)
+				)
+				(justify left)
+				(hide yes)
+			)
+		)

Commit message: Minor changes
Parts:
- R11: value 10 -> 0
Other:
- note added: "R10, R11 are zero-value resistors. Add appropriate resistors if you experience noise issues on the SPI lines."
Changed lines of the file:
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@@
+		)
+	)
+	(text "R10, R11 are zero-value resistors. \nAdd appropriate resistors if you \nexperience noise issues on the SPI lines."
+		(exclude_from_sim no)
+		(at 241.046 100.584 0)
+		(effects
+			(font
+				(size 1.27 1.27)
+			)
+			(justify left)
 		)
 	)
@@
 			)
 		)
-		(property "Value" "10"
+		(property "Value" "0"
 			(at 207.01 64.7699 0)
 			(effects
